Commit message: v1 type shit

File: robot_desc/robot.urdf (robot description, URDF)
Before this commit: robot my-robot, 8 links, 7 joints
Links:
- removed link danda_support_v5
- removed link danda_v4
- removed link fusioncomponent
- removed link fusioncomponent_2
- removed link fusioncomponent_3
- removed link fusioncomponent_4
- removed link fusioncomponent_5
- removed link fusioncomponent_6
- added link module_0_rod_main, mass 0.02; collision cylinder length=0.11 radius=0.006; visual mesh filename=../stls/danda_v4.stl
- added link module_0_rod_support, mass 0.02; collision cylinder length=0.11 radius=0.006; visual mesh filename=../stls/danda_support_v5.stl
- added link module_1_rod_main, mass 0.02; collision cylinder length=0.11 radius=0.006; visual mesh filename=../stls/danda_v4.stl
- added link module_1_rod_support, mass 0.02; collision cylinder length=0.11 radius=0.006; visual mesh filename=../stls/danda_support_v5.stl
- added link module_2_rod_main, mass 0.02; collision cylinder length=0.11 radius=0.006; visual mesh filename=../stls/danda_v4.stl
- added link module_2_rod_support, mass 0.02; collision cylinder length=0.11 radius=0.006; visual mesh filename=../stls/danda_support_v5.stl
- added link module_3_rod_main, mass 0.02; collision cylinder length=0.11 radius=0.006; visual mesh filename=../stls/danda_v4.stl
- added link module_3_rod_support, mass 0.02; collision cylinder length=0.11 radius=0.006; visual mesh filename=../stls/danda_support_v5.stl
- added link module_4_rod_main, mass 0.02; collision cylinder length=0.11 radius=0.006; visual mesh filename=../stls/danda_v4.stl
- added link module_4_rod_support, mass 0.02; collision cylinder length=0.11 radius=0.006; visual mesh filename=../stls/danda_support_v5.stl
- added link plate_0, mass 0.12; collision box size=0.12 0.12 0.016; visual mesh filename=../stls/fusioncomponent.stl
- added link plate_1, mass 0.12; collision box size=0.12 0.12 0.016; visual mesh filename=../stls/fusioncomponent.stl
- added link plate_2, mass 0.12; collision box size=0.12 0.12 0.016; visual mesh filename=../stls/fusioncomponent.stl
- added link plate_3, mass 0.12; collision box size=0.12 0.12 0.016; visual mesh filename=../stls/fusioncomponent.stl
- added link plate_4, mass 0.12; collision box size=0.12 0.12 0.016; visual mesh filename=../stls/fusioncomponent.stl
- added link plate_5, mass 0.12; collision box size=0.12 0.12 0.016; visual mesh filename=../stls/fusioncomponent.stl
Joints:
- removed joint 1
- removed joint 10
- removed joint 2
- removed joint 3
- removed joint 5
- removed joint 6
- removed joint 9
- added joint module_0_servo_a: type revolute, parent plate_0, child module_0_rod_main, origin xyz=0.028 -0.018 0 rpy=0 0 0, axis 0 0 1, limit lower=-1.0472 upper=1.0472 effort=12 velocity=4
- added joint module_0_servo_b: type revolute, parent module_0_rod_main, child plate_1, origin xyz=0 0 0.11 rpy=0 0 0, axis 1 0 0, limit lower=-1.0472 upper=1.0472 effort=12 velocity=4
- added joint module_0_support_fixed: type fixed, parent plate_0, child module_0_rod_support, origin xyz=-0.028 0.018 0 rpy=0 0 0
- added joint module_1_servo_a: type revolute, parent plate_1, child module_1_rod_main, origin xyz=0.028 -0.018 0 rpy=0 0 0, axis 0 0 1, limit lower=-1.0472 upper=1.0472 effort=12 velocity=4
- added joint module_1_servo_b: type revolute, parent module_1_rod_main, child plate_2, origin xyz=0 0 0.11 rpy=0 0 0, axis 1 0 0, limit lower=-1.0472 upper=1.0472 effort=12 velocity=4
- added joint module_1_support_fixed: type fixed, parent plate_1, child module_1_rod_support, origin xyz=-0.028 0.018 0 rpy=0 0 0
- added joint module_2_servo_a: type revolute, parent plate_2, child module_2_rod_main, origin xyz=0.028 -0.018 0 rpy=0 0 0, axis 0 0 1, limit lower=-1.0472 upper=1.0472 effort=12 velocity=4
- added joint module_2_servo_b: type revolute, parent module_2_rod_main, child plate_3, origin xyz=0 0 0.11 rpy=0 0 0, axis 1 0 0, limit lower=-1.0472 upper=1.0472 effort=12 velocity=4
- added joint module_2_support_fixed: type fixed, parent plate_2, child module_2_rod_support, origin xyz=-0.028 0.018 0 rpy=0 0 0
- added joint module_3_servo_a: type revolute, parent plate_3, child module_3_rod_main, origin xyz=0.028 -0.018 0 rpy=0 0 0, axis 0 0 1, limit lower=-1.0472 upper=1.0472 effort=12 velocity=4
- added joint module_3_servo_b: type revolute, parent module_3_rod_main, child plate_4, origin xyz=0 0 0.11 rpy=0 0 0, axis 1 0 0, limit lower=-1.0472 upper=1.0472 effort=12 velocity=4
- added joint module_3_support_fixed: type fixed, parent plate_3, child module_3_rod_support, origin xyz=-0.028 0.018 0 rpy=0 0 0
- added joint module_4_servo_a: type revolute, parent plate_4, child module_4_rod_main, origin xyz=0.028 -0.018 0 rpy=0 0 0, axis 0 0 1, limit lower=-1.0472 upper=1.0472 effort=12 velocity=4
- added joint module_4_servo_b: type revolute, parent module_4_rod_main, child plate_5, origin xyz=0 0 0.11 rpy=0 0 0, axis 1 0 0, limit lower=-1.0472 upper=1.0472 effort=12 velocity=4
- added joint module_4_support_fixed: type fixed, parent plate_4, child module_4_rod_support, origin xyz=-0.028 0.018 0 rpy=0 0 0
